File: cc2652p2-tcp.brd (EAGLE design)
At the start: 62 x 40 mm, 27 parts, among them J1 629105150921, J2 61300611821, U1 CC2652P2-DUOWEISI, U2 AP2112K, U3 USR-K6

Commit message: tests with ESP-01
Parts:
- removed C5: 100n, rcl:C0805
- removed R4, R5: 10k, rcl:R0805
- removed U$3: ESP-01, ESP-01:ESP-01
- moved U$5 35.1 mm to (52.0, 25.5)
- moved U$6 28.5 mm to (46.6, 20.9)
- renumbered USR-RST to RST
Connections:
- removed net N$8: R4.2, U$3.3
- removed net N$9: R5.2, U$3.5
- net GND: no longer C5.2, U$3.7
- net RXD: no longer U$3.8
- net TXD: no longer U$3.1
- net VCC: no longer C5.1, R4.1, R5.1, U$3.2
Routing:
- net VCC: track 101.9 -> 71.8 mm, vias 3 -> 2
- net RXD: track 53.8 -> 26.4 mm
- net TXD: track 47.4 -> 25.9 mm
- net N$8: track 3.41 -> 0.00 mm
- net N$9: track 3.27 -> 0.00 mm
Other:
- board text added: "5s to factory reset ethernet module"
- board text removed: "1"
- board text removed: "100nF"
- board text removed: "10k"
- board text removed: "ESP-01"
- board text removed: "push 5s to factory reset the ethernet module"
- board text removed: "when using ESP populate C5, R4, R5"

Commit message: tests with ESP-01
Parts:
- added C5: 100n, rcl:C0805
- added R4, R5, R6: 10k, rcl:R0805
- added U$3: ESP-01, ESP-01:ESP-01
- moved U$5 35.1 mm to (17.0, 23.5)
- moved U$6 28.5 mm to (19.6, 11.9)
Connections:
- new net N$7: R5.2, U$3.6
- new net N$8: R6.2, U$3.3
- net GND: now also C5.2, U$3.7
- net N$1: now also R4.2, U$3.4
- net RXD: now also U$3.8
- net TXD: now also U$3.1
- net VCC: now also C5.1, R4.1, R5.1, R6.1, U$3.2
Routing:
- net RXD: track 26.4 -> 58.4 mm
- net N$1: track 8.52 -> 38.6 mm
- net VCC: track 71.8 -> 100.5 mm, vias 2 -> 3
- net TXD: track 25.9 -> 47.4 mm
- net N$7: track 0.00 -> 6.00 mm
Other:
- board text added: "1"
- board text added: "100nF"
- board text added: "10k"
- board text added: "5s to factory reset ethernet module / ESP-01 reset"
- board text added: "ESP-01"
- board text added: "when using ESP populate C5 (100nF), R4-R6 (10k)"
- board text removed: "5s to factory reset ethernet module"

Commit message: removed ESP-01
Parts:
- removed C5: 100n, rcl:C0805
- removed R4, R5, R6: 10k, rcl:R0805
- removed U$3: ESP-01, ESP-01:ESP-01
- moved U$5 35.1 mm to (52.0, 25.5)
- moved U$6 28.5 mm to (46.6, 20.9)
Connections:
- removed net N$7: R5.2, U$3.6
- removed net N$8: R6.2, U$3.3
- net GND: no longer C5.2, U$3.7
- net N$1: no longer R4.2, U$3.4
- net RXD: no longer U$3.8
- net TXD: no longer U$3.1
- net VCC: no longer C5.1, R4.1, R5.1, R6.1, U$3.2
Routing:
- net RXD: track 58.4 -> 26.4 mm
- net N$1: track 38.6 -> 8.52 mm
- net VCC: track 100.5 -> 71.8 mm, vias 3 -> 2
- net TXD: track 47.4 -> 25.9 mm
- net N$7: track 6.00 -> 0.00 mm
Other:
- board text added: "5s to factory reset ethernet module"
- board text removed: "1"
- board text removed: "100nF"
- board text removed: "10k"
- board text removed: "5s to factory reset ethernet module / ESP-01 reset"
- board text removed: "ESP-01"
- board text removed: "when using ESP populate C5 (100nF), R4-R6 (10k)"

Commit message: V0.2
Parts:
- C4: value 22u -> 22 µF; device rcl:PANASONIC_C -> Eagle_WCAP-ASLL (rev20a):WCAP-ASLL_5X5.5(DXL)
- renumbered RST to USR-RST
Connections:
- net +5V: now also C4.1; no longer C4.+
- net GND: now also C4.2; no longer C4.-
Changed lines of the file:
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@@
 </layers>
 <board>
-<fusionsync huburn="a.cGVyc29uYWw6dWUyYzE1ODk4" projecturn="a.cGVyc29uYWw6dWUyYzE1ODk4IzIwMTkwNTIyMTk1MjcwNTc2" f3durn="urn:adsk.wipprod:dm.lineage:9xs_leqXRNeERXO3xgMQjw" pcbguid="" lastpulledtime="" lastsyncedchangeguid="" latestrevisionid="72b46ca4-16e5-4294-894f-9f9710218d27" lastsyncedrevisionid="72b46ca4-16e5-4294-894f-9f9710218d27" lastboardhashguid="4ccfb380-aebb-dbf3-aaab-a7c79df8eed3" lastpushedtime="2022-03-14T15:44:54Z" linktopcb3d="true"/>
+<fusionsync huburn="a.cGVyc29uYWw6dWUyYzE1ODk4" projecturn="a.cGVyc29uYWw6dWUyYzE1ODk4IzIwMTkwNTIyMTk1MjcwNTc2" f3durn="urn:adsk.wipprod:dm.lineage:9xs_leqXRNeERXO3xgMQjw" pcbguid="" lastpulledtime="" lastsyncedchangeguid="" latestrevisionid="d605f5ff-106c-4ada-a552-63e0fda9a90d" lastsyncedrevisionid="d605f5ff-106c-4ada-a552-63e0fda9a90d" lastboardhashguid="ce96a2d2-63ee-c4ce-8285-3bafe0439aab" lastpushedtime="2022-03-21T12:38:21Z" linktopcb3d="true"/>
 <plain>
 <text x="55.2" y="6.8" size="1.27" layer="26" rot="MR0">CC2652P2 TCP
@@
 <hole x="58" y="37" drill="3"/>
 <hole x="58" y="3" drill="3"/>
-<text x="39.8" y="15.3" size="0.8128" layer="25" font="vector" ratio="12" align="center">5s to factory reset
+<text x="39.8" y="15" size="0.8128" layer="25" font="vector" ratio="12" align="center">5s to factory reset
 ethernet module</text>
 <text x="6" y="20" size="1.4224" layer="26" font="vector" ratio="11" rot="MR270" align="center">Based on an idea from
@@
 <element name="U1" library="codm" library_urn="urn:adsk.eagle:library:11602856" package="CC2652P2-DUOWEISI" package3d_urn="urn:adsk.eagle:package:27394862/7" value="CC2652P2-DUOWEISI" x="19.5" y="32.8" smashed="yes" rot="R180"/>
 <element name="C2" library="rcl" library_urn="urn:adsk.eagle:library:334" package="C0805" package3d_urn="urn:adsk.eagle:package:23617/2" value="1u" x="45.9" y="12.6" smashed="yes">
-<attribute name="NAME" x="48.0984" y="12.6" size="0.8128" layer="25" align="center-left"/>
+<attribute name="NAME" x="45.9" y="13.7354" size="0.8128" layer="25" align="bottom-center"/>
 <attribute name="POPULARITY" value="88" x="41.9" y="19.6" size="1.778" layer="27" display="off"/>
 <attribute name="SPICEPREFIX" value="C" x="41.9" y="19.6" size="1.778" layer="27" display="off"/>
@@
 </element>
 <element name="C3" library="rcl" library_urn="urn:adsk.eagle:library:334" package="C0805" package3d_urn="urn:adsk.eagle:package:23617/2" value="1u" x="45.9" y="6.6" smashed="yes" rot="R180">
-<attribute name="NAME" x="48.0984" y="6.6" size="0.8128" layer="25" align="center-left"/>
+<attribute name="NAME" x="45.9" y="5.4646" size="0.8128" layer="25" align="top-center"/>
 <attribute name="POPULARITY" value="88" x="45.9" y="6.6" size="1.778" layer="27" rot="R180" display="off"/>
 <attribute name="SPICEPREFIX" value="C" x="45.9" y="6.6" size="1.778" layer="27" rot="R180" display="off"/>
@@
 <attribute name="NAME" x="30.025" y="18.27" size="0.8128" layer="21" font="vector" rot="R180" align="center"/>
 </element>
-<element name="C4" library="rcl" library_urn="urn:adsk.eagle:library:334" package="PANASONIC_C" package3d_urn="urn:adsk.eagle:package:23422/2" value="22u" x="51.9" y="9.6" smashed="yes" rot="R90">
-<attribute name="NAME" x="51.9" y="13.377" size="0.8128" layer="25" align="bottom-center"/>
-<attribute name="SPICEPREFIX" value="C" x="31.9" y="1.6" size="1.778" layer="27" rot="R90" display="off"/>
-<attribute name="VALUE" x="55.675" y="6.95" size="1.016" layer="27" rot="R90"/>
+<element name="C4" library="Eagle_WCAP-ASLL (rev20a)" package="WCAP-ASLL_5X5.5(DXL)" package3d_urn="urn:adsk.eagle:package:18354036/2" value="22  µF " x="51.9" y="9.6" smashed="yes" rot="R90">
+<attribute name="DATASHEET-URL" value="https://www.we-online.com/catalog/datasheet/865060342002.pdf" x="51.9" y="9.6" size="1.778" layer="27" rot="R90" display="off"/>
+<attribute name="DF" value="16%" x="51.9" y="9.6" size="1.778" layer="27" rot="R90" display="off"/>
+<attribute name="DIAMETER" value="5mm" x="51.9" y="9.6" size="1.778" layer="27" rot="R90" display="off"/>
+<attribute name="I-LEAK" value="3.52uA" x="51.9" y="9.6" size="1.778" layer="27" rot="R90" display="off"/>
+<attribute name="I-RIPPLE" value="150mA" x="51.9" y="9.6" size="1.778" layer="27" rot="R90" display="off"/>
+<attribute name="L" value="5.5mm" x="51.9" y="9.6" size="1.778" layer="27" rot="R90" display="off"/>
+<attribute name="NAME" x="51.9" y="13.677" size="0.8128" layer="25" align="bottom-center"/>
+<attribute name="OPERATING-TEMPERATURE" value="-55 °C up to +105 °C" x="51.9" y="9.6" size="1.778" layer="27" rot="R90" display="off"/>
+<attribute name="PART-NUMBER" value=" 865060342002 " x="51.9" y="9.6" size="1.778" layer="27" rot="R90" display="off"/>
+<attribute name="TECHNICAL-REFERENCE" value="ASEC055220M016DVCTBB000" x="51.9" y="9.6" size="1.778" layer="27" rot="R90" display="off"/>
+<attribute name="VALUE" value="22  µF " x="55.675" y="6.95" size="1.016" layer="27" rot="R90"/>
+<attribute name="VR" value="16V(DC)" x="51.9" y="9.6" size="1.778" layer="27" rot="R90" display="off"/>
+<attribute name="Z" value="0.8Ohm" x="51.9" y="9.6" size="1.778" layer="27" rot="R90" display="off"/>
 </element>
 <element name="J1" library="codm" library_urn="urn:adsk.eagle:library:11602856" package="629105150921" package3d_urn="urn:adsk.eagle:package:34282692/1" value="629105150921" x="60.2" y="9.8" smashed="yes" rot="R90">
@@
 <attribute name="VALUE" x="23.66" y="27.535" size="1.27" layer="27" rot="R270"/>
 </element>
-<element name="RST" library="434153017835_Eagle_WS-TASV_rev20a" package="434153017835" package3d_urn="urn:adsk.eagle:package:18304352/2" value="" x="39.8" y="11.5" smashed="yes">
+<element name="USR-RST" library="434153017835_Eagle_WS-TASV_rev20a" package="434153017835" package3d_urn="urn:adsk.eagle:package:18304352/2" value="" x="39.8" y="11.5" smashed="yes">
 <attribute name="DATASHEET-URL" value="https://www.we-online.com/catalog/datasheet/434153017835.pdf" x="39.8" y="11.5" size="0.8128" layer="27" font="vector" display="off"/>
 <attribute name="H" value="1.7mm" x="39.8" y="11.5" size="0.8128" layer="27" font="vector" display="off"/>
@@
 <contactref element="U2" pad="2"/>
 <contactref element="C1" pad="1"/>
-<contactref element="C4" pad="-"/>
+<contactref element="C4" pad="2"/>
 <contactref element="U3" pad="GND@1"/>
 <contactref element="U3" pad="GND@2"/>
@@
 <contactref element="LED1" pad="1"/>
 <contactref element="RESET" pad="4"/>
-<contactref element="RST" pad="4"/>
+<contactref element="USR-RST" pad="4"/>
 </signal>
 <signal name="RXD">
@@
 <contactref element="U2" pad="1"/>
 <contactref element="U2" pad="3"/>
-<contactref element="C4" pad="+"/>
+<contactref element="C4" pad="1"/>
 <wire x1="46.85" y1="12.6" x2="50.95" y2="12.6" width="0.254" layer="1"/>
-<wire x1="50.95" y1="12.6" x2="51.9" y2="11.65" width="0.254" layer="1"/>
+<wire x1="50.95" y1="12.6" x2="51.9" y2="11.8" width="0.254" layer="1"/>
 <wire x1="46.85" y1="12.6" x2="46.85" y2="10.9001" width="0.254" layer="1"/>
 <wire x1="46.85" y1="10.9001" x2="47.2001" y2="10.55" width="0.254" layer="1"/>
@@
 <wire x1="46.45" y1="8.65" x2="47.2001" y2="8.65" width="0.254" layer="1"/>
 <contactref element="J1" pad="1"/>
-<wire x1="51.9" y1="11.65" x2="55.05" y2="8.5" width="0.254" layer="1"/>
+<wire x1="51.9" y1="11.8" x2="55.05" y2="8.5" width="0.254" layer="1"/>
 <wire x1="55.05" y1="8.5" x2="57.865" y2="8.5" width="0.254" layer="1"/>
 </signal>
@@
 <signal name="N$1">
 <contactref element="U3" pad="6"/>
-<contactref element="RST" pad="1"/>
+<contactref element="USR-RST" pad="1"/>
 <wire x1="38.125" y1="12.225" x2="38.125" y2="20.3446" width="0.1524" layer="1"/>
 <wire x1="38.125" y1="20.3446" x2="37.8412" y2="20.6284" width="0.1524" layer="1"/>

Commit message: V0.2
Parts:
- R2, R3: value 1k -> 2k7
Changed lines of the file:
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@@
 <attribute name="VALUE" x="47.04" y="3.44" size="0.4064" layer="27" rot="R180" align="bottom-center"/>
 </element>
-<element name="R2" library="rcl" library_urn="urn:adsk.eagle:library:334" package="R0805" package3d_urn="urn:adsk.eagle:package:23553/2" value="1k" x="26.2" y="31" smashed="yes" rot="R270">
+<element name="R2" library="rcl" library_urn="urn:adsk.eagle:library:334" package="R0805" package3d_urn="urn:adsk.eagle:package:23553/2" value="2k7" x="26.2" y="31" smashed="yes" rot="R270">
 <attribute name="NAME" x="26.2" y="33.1254" size="0.8128" layer="25" align="bottom-center"/>
 <attribute name="POPULARITY" value="86" x="26.2" y="31" size="1.778" layer="27" rot="R270" display="off"/>
@@
 <attribute name="VALUE" x="23.66" y="31.635" size="1.27" layer="27" rot="R270"/>
 </element>
-<element name="R3" library="rcl" library_urn="urn:adsk.eagle:library:334" package="R0805" package3d_urn="urn:adsk.eagle:package:23553/2" value="1k" x="26.2" y="26.9" smashed="yes" rot="R270">
+<element name="R3" library="rcl" library_urn="urn:adsk.eagle:library:334" package="R0805" package3d_urn="urn:adsk.eagle:package:23553/2" value="2k7" x="26.2" y="26.9" smashed="yes" rot="R270">
 <attribute name="NAME" x="26.2" y="24.7746" size="0.8128" layer="25" align="top-center"/>
 <attribute name="POPULARITY" value="86" x="26.2" y="26.9" size="1.778" layer="27" rot="R270" display="off"/>
