File: cc2652p2-tcp.sch (EAGLE design)
At the start: 23 parts, among them J1 629105150921, J2 61300611821, U1 CC2652P2-DUOWEISI, U2 AP2112K, U3 USR-K6

Commit message: removed ESP-01
Parts:
- removed C5: 100n, rcl:C-EUC0805
- removed R4, R5, R6: 10k, rcl:R-EU_R0805
- removed U$3: ESP-01, ESP-01:ESP-01
Connections:
- removed net N$7: R5.2, U$3.CH_PD
- removed net N$8: R6.2, U$3.IO0
- net GND: no longer C5.2, U$3.GND
- net N$1: no longer R4.2, U$3.RST
- net RXD: no longer U$3.TX
- net TXD: no longer U$3.RX
- net VCC: no longer C5.1, R4.1, R5.1, R6.1, U$3.VCC
Changed lines of the file:
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@@
 <part name="R2" library="rcl" library_urn="urn:adsk.eagle:library:334" deviceset="R-EU_" device="R0805" package3d_urn="urn:adsk.eagle:package:23553/2" value="1k"/>
 <part name="R3" library="rcl" library_urn="urn:adsk.eagle:library:334" deviceset="R-EU_" device="R0805" package3d_urn="urn:adsk.eagle:package:23553/2" value="1k"/>
-<part name="U$3" library="ESP-01" deviceset="ESP-01" device="" override_package3d_urn="urn:adsk.eagle:package:34247119/2" override_package_urn="urn:adsk.eagle:footprint:34247120/1"/>
-<part name="GND5" library="supply1" deviceset="GND" device=""/>
-<part name="P+3" library="supply1" library_urn="urn:adsk.eagle:library:371" deviceset="VCC" device=""/>
-<part name="C5" library="rcl" library_urn="urn:adsk.eagle:library:334" deviceset="C-EU" device="C0805" package3d_urn="urn:adsk.eagle:package:23617/2" value="100n"/>
-<part name="R4" library="rcl" library_urn="urn:adsk.eagle:library:334" deviceset="R-EU_" device="R0805" package3d_urn="urn:adsk.eagle:package:23553/2" value="10k"/>
-<part name="R5" library="rcl" library_urn="urn:adsk.eagle:library:334" deviceset="R-EU_" device="R0805" package3d_urn="urn:adsk.eagle:package:23553/2" value="10k"/>
 <part name="RST" library="434153017835_Eagle_WS-TASV_rev20a" deviceset="434153017835" device="" package3d_urn="urn:adsk.eagle:package:18304352/2"/>
-<part name="R6" library="rcl" library_urn="urn:adsk.eagle:library:334" deviceset="R-EU_" device="R0805" package3d_urn="urn:adsk.eagle:package:23553/2" value="10k"/>
 </parts>
 <sheets>
@@
 <attribute name="VALUE" x="80.01" y="135.382" size="1.778" layer="96" rot="R180"/>
 </instance>
-<instance part="U$3" gate="G$1" x="223.52" y="124.46" smashed="yes">
-<attribute name="NAME" x="217.17" y="132.715" size="1.778" layer="95"/>
-</instance>
-<instance part="GND5" gate="1" x="208.28" y="111.76" smashed="yes">
-<attribute name="VALUE" x="205.74" y="109.22" size="1.778" layer="96"/>
-</instance>
-<instance part="P+3" gate="VCC" x="254" y="152.4" smashed="yes">
-<attribute name="VALUE" x="251.46" y="149.86" size="1.778" layer="96" rot="R90"/>
-</instance>
-<instance part="C5" gate="G$1" x="254" y="124.46" smashed="yes">
-<attribute name="NAME" x="255.524" y="124.841" size="1.778" layer="95"/>
-<attribute name="VALUE" x="255.524" y="119.761" size="1.778" layer="96"/>
-</instance>
-<instance part="R4" gate="G$1" x="243.84" y="137.16" smashed="yes" rot="R270">
-<attribute name="VALUE" x="240.538" y="140.97" size="1.778" layer="96" rot="R270"/>
-</instance>
-<instance part="R5" gate="G$1" x="248.92" y="137.16" smashed="yes" rot="R270">
-<attribute name="NAME" x="250.4186" y="140.97" size="1.778" layer="95" rot="R270"/>
-<attribute name="VALUE" x="245.618" y="140.97" size="1.778" layer="96" rot="R270"/>
-</instance>
 <instance part="RST" gate="G$1" x="198.12" y="55.88" smashed="yes" rot="R180">
 <attribute name="NAME" x="197.95" y="49.93" size="1.778" layer="95" rot="R180" align="bottom-center"/>
 <attribute name="VALUE" x="201.93" y="60.96" size="1.778" layer="96" rot="R180"/>
-</instance>
-<instance part="R6" gate="G$1" x="200.66" y="137.16" smashed="yes" rot="R270">
-<attribute name="NAME" x="202.1586" y="140.97" size="1.778" layer="95" rot="R270"/>
-<attribute name="VALUE" x="197.358" y="140.97" size="1.778" layer="96" rot="R270"/>
 </instance>
 </instances>
@@
 <wire x1="167.64" y1="119.38" x2="160.02" y2="119.38" width="0.1524" layer="91"/>
 <label x="160.02" y="119.38" size="1.4224" layer="95" rot="R180" xref="yes"/>
-</segment>
-<segment>
-<pinref part="U$3" gate="G$1" pin="VCC"/>
-<wire x1="238.76" y1="129.54" x2="254" y2="129.54" width="0.1524" layer="91"/>
-<pinref part="C5" gate="G$1" pin="1"/>
-<wire x1="254" y1="129.54" x2="254" y2="127" width="0.1524" layer="91"/>
-<pinref part="P+3" gate="VCC" pin="VCC"/>
-<wire x1="254" y1="129.54" x2="254" y2="144.78" width="0.1524" layer="91"/>
-<junction x="254" y="129.54"/>
-<wire x1="254" y1="144.78" x2="254" y2="149.86" width="0.1524" layer="91"/>
-<pinref part="R4" gate="G$1" pin="1"/>
-<wire x1="243.84" y1="144.78" x2="243.84" y2="142.24" width="0.1524" layer="91"/>
-<wire x1="243.84" y1="144.78" x2="248.92" y2="144.78" width="0.1524" layer="91"/>
-<junction x="254" y="144.78"/>
-<pinref part="R5" gate="G$1" pin="1"/>
-<wire x1="248.92" y1="144.78" x2="254" y2="144.78" width="0.1524" layer="91"/>
-<wire x1="248.92" y1="142.24" x2="248.92" y2="144.78" width="0.1524" layer="91"/>
-<junction x="248.92" y="144.78"/>
-<pinref part="R6" gate="G$1" pin="1"/>
-<wire x1="200.66" y1="142.24" x2="200.66" y2="144.78" width="0.1524" layer="91"/>
-<wire x1="200.66" y1="144.78" x2="243.84" y2="144.78" width="0.1524" layer="91"/>
-<junction x="243.84" y="144.78"/>
 </segment>
 </net>
@@
 <wire x1="160.02" y1="124.46" x2="167.64" y2="124.46" width="0.1524" layer="91"/>
 </segment>
-<segment>
-<pinref part="U$3" gate="G$1" pin="GND"/>
-<wire x1="210.82" y1="121.92" x2="208.28" y2="121.92" width="0.1524" layer="91"/>
-<pinref part="GND5" gate="1" pin="GND"/>
-<wire x1="208.28" y1="121.92" x2="208.28" y2="116.84" width="0.1524" layer="91"/>
-<pinref part="C5" gate="G$1" pin="2"/>
-<wire x1="208.28" y1="116.84" x2="208.28" y2="114.3" width="0.1524" layer="91"/>
-<wire x1="254" y1="119.38" x2="254" y2="116.84" width="0.1524" layer="91"/>
-<wire x1="254" y1="116.84" x2="208.28" y2="116.84" width="0.1524" layer="91"/>
-<junction x="208.28" y="116.84"/>
-</segment>
 </net>
 <net name="RXD" class="0">
@@
 <label x="160.02" y="116.84" size="1.4224" layer="95" rot="R180" xref="yes"/>
 </segment>
-<segment>
-<pinref part="U$3" gate="G$1" pin="TX"/>
-<wire x1="238.76" y1="121.92" x2="241.3" y2="121.92" width="0.1524" layer="91"/>
-<label x="241.3" y="121.92" size="1.27" layer="95" xref="yes"/>
-</segment>
 </net>
 <net name="TXD" class="0">
@@
 <wire x1="167.64" y1="114.3" x2="160.02" y2="114.3" width="0.1524" layer="91"/>
 <label x="160.02" y="114.3" size="1.4224" layer="95" rot="R180" xref="yes"/>
-</segment>
-<segment>
-<pinref part="U$3" gate="G$1" pin="RX"/>
-<wire x1="210.82" y1="129.54" x2="208.28" y2="129.54" width="0.1524" layer="91"/>
-<label x="208.28" y="129.54" size="1.27" layer="95" rot="R180" xref="yes"/>
 </segment>
 </net>
@@
 <junction x="220.98" y="50.8"/>
 <wire x1="220.98" y1="68.58" x2="243.84" y2="68.58" width="0.1524" layer="91"/>
-<pinref part="R4" gate="G$1" pin="2"/>
-<wire x1="243.84" y1="132.08" x2="243.84" y2="127" width="0.1524" layer="91"/>
-<pinref part="U$3" gate="G$1" pin="RST"/>
-<wire x1="243.84" y1="127" x2="238.76" y2="127" width="0.1524" layer="91"/>
-<wire x1="243.84" y1="68.58" x2="243.84" y2="127" width="0.1524" layer="91"/>
-<junction x="243.84" y="127"/>
-</segment>
-</net>
-<net name="N$7" class="0">
-<segment>
-<pinref part="R5" gate="G$1" pin="2"/>
-<wire x1="248.92" y1="132.08" x2="248.92" y2="124.46" width="0.1524" layer="91"/>
-<pinref part="U$3" gate="G$1" pin="CH_PD"/>
-<wire x1="248.92" y1="124.46" x2="238.76" y2="124.46" width="0.1524" layer="91"/>
-</segment>
-</net>
-<net name="N$8" class="0">
-<segment>
-<pinref part="R6" gate="G$1" pin="2"/>
-<wire x1="200.66" y1="132.08" x2="200.66" y2="127" width="0.1524" layer="91"/>
-<pinref part="U$3" gate="G$1" pin="IO0"/>
-<wire x1="200.66" y1="127" x2="210.82" y2="127" width="0.1524" layer="91"/>
-</segment>
-</net>
+</segment>
+</net>

Commit message: V0.2
Parts:
- C4: value 22u -> 22 µF; device rcl:CPOL-EUC -> Eagle_WCAP-ASLL (rev20a):WCAP-ASLL_5X5.5_865060342002
- renumbered RST to USR-RST
Changed lines of the file:
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@@
 <part name="C1" library="rcl" library_urn="urn:adsk.eagle:library:334" deviceset="C-EU" device="C0805" package3d_urn="urn:adsk.eagle:package:23617/2" value="100n"/>
 <part name="U3" library="codm" library_urn="urn:adsk.eagle:library:11602856" deviceset="USR-K6" device="" package3d_urn="urn:adsk.eagle:package:34184974/12"/>
-<part name="C4" library="rcl" library_urn="urn:adsk.eagle:library:334" deviceset="CPOL-EU" device="C" package3d_urn="urn:adsk.eagle:package:23422/2" value="22u"/>
+<part name="C4" library="Eagle_WCAP-ASLL (rev20a)" deviceset="WCAP-ASLL_5X5.5" device="" package3d_urn="urn:adsk.eagle:package:18354036/2" technology="_865060342002" value="22  µF "/>
 <part name="J1" library="codm" library_urn="urn:adsk.eagle:library:11602856" deviceset="629105150921" device="" package3d_urn="urn:adsk.eagle:package:34282692/1" value="629105150921"/>
 <part name="GND2" library="supply1" deviceset="GND" device=""/>
@@
 <part name="R2" library="rcl" library_urn="urn:adsk.eagle:library:334" deviceset="R-EU_" device="R0805" package3d_urn="urn:adsk.eagle:package:23553/2" value="1k"/>
 <part name="R3" library="rcl" library_urn="urn:adsk.eagle:library:334" deviceset="R-EU_" device="R0805" package3d_urn="urn:adsk.eagle:package:23553/2" value="1k"/>
-<part name="RST" library="434153017835_Eagle_WS-TASV_rev20a" deviceset="434153017835" device="" package3d_urn="urn:adsk.eagle:package:18304352/2"/>
+<part name="USR-RST" library="434153017835_Eagle_WS-TASV_rev20a" deviceset="434153017835" device="" package3d_urn="urn:adsk.eagle:package:18304352/2"/>
 </parts>
 <sheets>
@@
 </instance>
 <instance part="U3" gate="G$1" x="246.38" y="48.26" smashed="yes"/>
-<instance part="C4" gate="G$1" x="73.66" y="25.4" smashed="yes">
-<attribute name="NAME" x="74.803" y="25.8826" size="1.778" layer="95"/>
-<attribute name="VALUE" x="74.803" y="20.8026" size="1.778" layer="96"/>
+<instance part="C4" gate="G$1" x="73.66" y="22.86" smashed="yes" rot="R90">
+<attribute name="NAME" x="73.1774" y="24.003" size="1.778" layer="95" rot="R90"/>
+<attribute name="VALUE" x="78.2574" y="24.003" size="1.778" layer="96" rot="R90"/>
 </instance>
 <instance part="J1" gate="G$1" x="60.96" y="45.72" smashed="yes" rot="R90">
@@
 <attribute name="VALUE" x="80.01" y="135.382" size="1.778" layer="96" rot="R180"/>
 </instance>
-<instance part="RST" gate="G$1" x="198.12" y="55.88" smashed="yes" rot="R180">
+<instance part="USR-RST" gate="G$1" x="198.12" y="55.88" smashed="yes" rot="R180">
 <attribute name="NAME" x="197.95" y="49.93" size="1.778" layer="95" rot="R180" align="bottom-center"/>
 <attribute name="VALUE" x="201.93" y="60.96" size="1.778" layer="96" rot="R180"/>
@@
 <junction x="220.98" y="33.02"/>
 <wire x1="190.5" y1="33.02" x2="190.5" y2="58.42" width="0.1524" layer="91"/>
-<pinref part="RST" gate="G$1" pin="4"/>
+<pinref part="USR-RST" gate="G$1" pin="4"/>
 <wire x1="190.5" y1="58.42" x2="193.04" y2="58.42" width="0.1524" layer="91"/>
 </segment>
@@
 <segment>
 <pinref part="U3" gate="G$1" pin="CFG"/>
-<pinref part="RST" gate="G$1" pin="1"/>
+<pinref part="USR-RST" gate="G$1" pin="1"/>
 <wire x1="228.6" y1="50.8" x2="220.98" y2="50.8" width="0.1524" layer="91"/>
 <wire x1="220.98" y1="50.8" x2="203.2" y2="50.8" width="0.1524" layer="91"/>

Commit message: V0.2
Parts:
- R2, R3: value 1k -> 2k7
Changed lines of the file:
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@@
 <part name="LED1" library="Eagle_WL-SMCW (rev22a)" deviceset="WL-SMCW_0805" device="" package3d_urn="urn:adsk.eagle:package:19028167/3" technology="_150080GS75000" value="150080GS75000"/>
 <part name="LED2" library="Eagle_WL-SMCW (rev22a)" deviceset="WL-SMCW_0805" device="" package3d_urn="urn:adsk.eagle:package:19028167/3" technology="_150080RS75000" value="150080RS75000"/>
-<part name="R2" library="rcl" library_urn="urn:adsk.eagle:library:334" deviceset="R-EU_" device="R0805" package3d_urn="urn:adsk.eagle:package:23553/2" value="1k"/>
-<part name="R3" library="rcl" library_urn="urn:adsk.eagle:library:334" deviceset="R-EU_" device="R0805" package3d_urn="urn:adsk.eagle:package:23553/2" value="1k"/>
+<part name="R2" library="rcl" library_urn="urn:adsk.eagle:library:334" deviceset="R-EU_" device="R0805" package3d_urn="urn:adsk.eagle:package:23553/2" value="2k7"/>
+<part name="R3" library="rcl" library_urn="urn:adsk.eagle:library:334" deviceset="R-EU_" device="R0805" package3d_urn="urn:adsk.eagle:package:23553/2" value="2k7"/>
 <part name="USR-RST" library="434153017835_Eagle_WS-TASV_rev20a" deviceset="434153017835" device="" package3d_urn="urn:adsk.eagle:package:18304352/2"/>
 </parts>
